Commit message: Fix Gazebo Harmonic simulation with working sensors and robot control

File: cowbot_ws/src/cowbot_description/onshape/cowbot.xacro (robot description, xacro)
@@ -98,5 +98,5 @@
       <parent link="${robot_name}_motor_1"/>
       <child link="${robot_name}_wheel_right"/>
-      <axis xyz="0 0 1"/>
+      <axis xyz="0 0 -1"/>
     </joint>
     <!-- Joint from base_link to motor_1 -->
@@ -176,9 +176,9 @@
       <parent link="${robot_name}_motor_2"/>
       <child link="${robot_name}_wheel_left"/>
-      <axis xyz="0 0 -1"/>
+      <axis xyz="0 0 1"/>
     </joint>
     <!-- Joint from base_link to motor_2 -->
     <joint name="${robot_name}_left_motor" type="fixed">
-      <origin xyz="0.069556 -0.0408289 0.0260952" rpy="1.5708 0 0"/>
+      <origin xyz="-0.078444 0.0408289 0.0260952" rpy="1.5708 0 0"/>
       <parent link="${robot_name}_base_link"/>
       <child link="${robot_name}_motor_2"/>
@@ -211,5 +211,5 @@
     <!-- Joint from base_link to ball_caster -->
     <joint name="${robot_name}_caster" type="fixed">
-      <origin xyz="5.59691e-05 -0.0241949 0.00334516" rpy="0 0 1.5708"/>
+      <origin xyz="0.08 -0.0241949 0.00334516" rpy="0 0 1.5708"/>
       <parent link="${robot_name}_base_link"/>
       <child link="${robot_name}_ball_caster"/>
@@ -272,5 +272,5 @@
     </link>
     <!-- Joint from base_link to camera -->
-    <joint name="${robot_name}_camera" type="fixed">
+    <joint name="${robot_name}_camera_joint" type="fixed">
       <origin xyz="0.021056 -0.0168289 0.088598" rpy="1.5708 0 1.5708"/>
       <parent link="${robot_name}_base_link"/>

Commit message: Update: cowbot(xacro. urdf) and gazebo world

File: cowbot_ws/src/cowbot_description/onshape/cowbot.xacro (robot description, xacro)
@@ -189,7 +189,6 @@
       <inertial>
         <origin xyz="0 0 0" rpy="0 0 0"/>
-        <mass value="0.01"/>
-        <inertia ixx="1e-09" ixy="0" ixz="0" iyy="1e-09" iyz="0" izz="1e-09"/>
-      </inertial>
+        <mass value="0.05"/>
+        <inertia ixx="0.0001" ixy="0" ixz="0" iyy="0.0001" iyz="0" izz="0.0001"/> </inertial>
       <!-- Part pololu_ball_caster -->
       <visual>
